File: hotswap_rgb/dumbpad.kicad_pcb (KiCad board)
At the start: 2 copper layers, 97 x 78.5 mm, 62 parts

Commit message: new files I guess
Other:
- board text added: "Hotswap - Rgb - Smartpad"
- board text added: "Logan's Personalised Smartpad"
- board text added: "WayWayWay"
- board text added: "imchipwood x deveth0 x DwarvenFrogge"
- board text removed: "dumbpad - hotswap - rgb"
- board text removed: "github.com/imchipwood/dumbpad"
- board text removed: "imchipwood x deveth0"
